Commit message: Update SimulatedLab joint names and add robot controller GUI

File: SimulatedLab/urdf/SimulatedLab.urdf (robot description, URDF)
Before this commit: robot SimulatedLab, 9 links, 8 joints
Links:
- removed link base
- removed link base_link
- removed link robot-baseboard
- removed link slidebase
- removed link wrist
- added link MicroplateHolder, mass 0; collision mesh filename=package://SimulatedLab/meshes/MicroplateHolder.STL; visual mesh filename=package://SimulatedLab/meshes/MicroplateHolder.STL
- added link OpticalTable, mass 199.39; collision mesh filename=package://SimulatedLab/meshes/OpticalTable.STL; visual mesh filename=package://SimulatedLab/meshes/OpticalTable.STL
- added link Rail-Robot-connector, mass 0.55039; visual mesh filename=package://SimulatedLab/meshes/Rail-Robot-connector.STL
- added link SlideBrick, mass 0.41998; collision mesh filename=package://SimulatedLab/meshes/SlideBrick.STL; visual mesh filename=package://SimulatedLab/meshes/SlideBrick.STL
- added link SlideRail, mass 9.3221; collision mesh filename=package://SimulatedLab/meshes/SlideRail.STL; visual mesh filename=package://SimulatedLab/meshes/SlideRail.STL
- added link SquidMicroscope, mass 3.6417; collision mesh filename=package://SimulatedLab/meshes/SquidMicroscope.STL; visual mesh filename=package://SimulatedLab/meshes/SquidMicroscope.STL
- added link arm-base, mass 0.17228; visual mesh filename=package://SimulatedLab/meshes/arm-base.STL
- added link wrist1, mass 0.019467; visual mesh filename=package://SimulatedLab/meshes/wrist1.STL
- link arm1: mass 0.675270738615706 -> 0.67527; geometry visual mesh filename=package://SimulatedLab/meshes/arm1.STL
- link arm2: mass 0.271676187941207 -> 0.27168; geometry visual mesh filename=package://SimulatedLab/meshes/arm2.STL
- link arm3: mass 0.29343830579726 -> 0.29344
- link wrist2: mass 0.04637707880367 -> 0.010769; geometry visual mesh filename=package://SimulatedLab/meshes/wrist2.STL
Joints:
- removed joint arm1-2
- removed joint arm2-3
- removed joint base-arm
- removed joint fix2
- removed joint robot-base
- removed joint slide
- removed joint wrist1-2
- added joint Rail-Robot-connector-fix: type fixed, parent SlideBrick, child Rail-Robot-connector, origin xyz=-0.0041396 0.055847 0.072641 rpy=0 1.5708 0, axis 0 0 0
- added joint Slide: type prismatic, parent SlideRail, child SlideBrick, origin xyz=0.0041396 -0.033447 -0.7972 rpy=3.1416 0 0, axis 0 0 1, limit lower=-3.5 upper=0 effort=0 velocity=0
- added joint arm1J: type revolute, parent arm-base, child arm1, origin xyz=-0.0019527 0.047214 -0.051373 rpy=1.5708 -1.5708 -1.5708, axis 0 1 0, limit lower=-180 upper=180 effort=0 velocity=0
- added joint arm2J: type revolute, parent arm1, child arm2, origin xyz=0 0.19707 0.095476 rpy=-1.5675 0 0, axis 1 0 0, limit lower=-180 upper=180 effort=0 velocity=0
- added joint arm3J: type revolute, parent arm2, child arm3, origin xyz=0 0.2032 0 rpy=0.89363 0 0, axis 1 0 0, limit lower=-180 upper=180 effort=0 velocity=0
- added joint armbaseJ: type fixed, parent Rail-Robot-connector, child arm-base, origin xyz=0.0019527 -0.0078131 0.051373 rpy=0 0 0, axis 0 0 0
- added joint hotel-fix: type fixed, parent OpticalTable, child MicroplateHolder, origin xyz=0.818329937973544 -0.725482308658135 0.129836500776815 rpy=1.5707963267949 0 0, axis 0 0 0
- added joint microscope-fix: type fixed, parent OpticalTable, child SquidMicroscope, origin xyz=-0.073823 -0.66731 0.059932 rpy=1.5708 0 3.1416, axis 0 0 0
- added joint rail-fix: type fixed, parent OpticalTable, child SlideRail, origin xyz=0.14169 -1.1751 0.052089 rpy=-1.5708 0 -1.5708, axis 0 0 0
- added joint wrist2-j: type revolute, parent wrist1, child wrist2, origin xyz=0 0 0 rpy=0 0 0, axis 0 0.016592 0.99986, limit lower=-180 upper=180 effort=0 velocity=0, mimic joint=arm1J multiplier=1 offset=0
- joint arm-wrist: child wrist -> wrist1; limit (none) -> lower=-180 upper=180 effort=0 velocity=0; origin xyz=0 0 0.1524 rpy=0.76686 0 -3.1416 -> xyz=0 0 0.1524 rpy=2.35 0 3.1416; type continuous -> revolute

Commit message: Add collision geometry for arm-base and arm1 links, initialize simulation and execute example sequence

File: SimulatedLab/urdf/SimulatedLab.urdf (robot description, URDF)
Before this commit: robot SimulatedLab, 12 links, 11 joints
Links:
- link arm-base: geometry collision mesh filename=package://SimulatedLab/meshes/arm-base.STL; visual mesh filename=package://SimulatedLab/meshes/arm-base.STL
- link arm1: geometry collision mesh filename=package://SimulatedLab/meshes/arm1.STL; visual mesh filename=package://SimulatedLab/meshes/arm1.STL

Commit message: 🚀feat(SimulatedLab) add collision detection for wrist meshes🚀feat(test) initialize camera on simulation start

File: SimulatedLab/urdf/SimulatedLab.urdf (robot description, URDF)
Before this commit: robot SimulatedLab, 12 links, 11 joints
Links:
- link arm3: geometry visual mesh filename=package://SimulatedLab/meshes/arm3.STL
- link wrist1: geometry collision mesh filename=package://SimulatedLab/meshes/wrist1.STL; visual mesh filename=package://SimulatedLab/meshes/wrist1.STL
- link wrist2: geometry collision mesh filename=package://SimulatedLab/meshes/wrist2.STL; visual mesh filename=package://SimulatedLab/meshes/wrist2.STL
