Commit message: Fix joint names in dorna2-rebuild.yaml and update test.py for SimulatedLab robot

File: dorna2-rebuild/urdf/dorna2-rebuild.urdf (robot description, URDF)
Before this commit: robot dorna2-rebuild, 7 links, 6 joints
Links:
- removed link arm_base
- added link arm-base, mass 0.722677101161874; collision mesh filename=package://dorna2-rebuild/meshes/arm-base.STL; visual mesh filename=package://dorna2-rebuild/meshes/arm-base.STL
- link arm1: mass 0.67527 -> 0.675270731859809
- link arm2: mass 0.27168 -> 0.271676192230468
- link arm3: mass 0.29344 -> 0.293438315476537
- link gripper: mass 2.9259 -> 1.25
- link wrist1: mass 0.019467 -> 0.0194666574215483
- link wrist2: mass 0.010769 -> 0.0107694009383611
Joints:
- removed joint arm2j
- removed joint arm3j
- removed joint wrist1j
- removed joint wrist2j
- added joint arm2-j: type revolute, parent arm1, child arm2, origin xyz=-0.095476 0 0.17761 rpy=0 0 0, axis 0 -1 0, limit lower=-91 upper=181 effort=0 velocity=0
- added joint arm3-j: type revolute, parent arm2, child arm3, origin xyz=-0.2032 0.0009058 0 rpy=0 0 0, axis 0 -1 0, limit lower=-142 upper=142 effort=0 velocity=0
- added joint wrist1-j: type revolute, parent arm3, child wrist1, origin xyz=-0.1524 -0.0010033 0 rpy=0 0.016592 0, axis 0 1 0, limit lower=-135 upper=135 effort=0 velocity=0
- added joint wrist2-j: type revolute, parent wrist1, child wrist2, origin xyz=0 0 0 rpy=0 0 0, axis -0.99986 0 -0.016592, limit lower=-360 upper=360 effort=0 velocity=0
- joint arm1j: axis 0 1 0 -> 0 0 1; origin xyz=0.012824 -0.0009058 0 rpy=1.5708 0 -1.5708 -> xyz=0.012824 -0.0009058 0 rpy=0 0 0; parent arm_base -> arm-base
- joint gripper-j: origin xyz=0.019031 -0.015038 0.086123 rpy=-0.016592 3.1072E-05 0.0018725 -> xyz=0.021303 -2.739 -1.0897 rpy=-0.0018728 -0.016592 0
