Commit message: 🚀feat(URDF): update mesh filenames 🛠️refactor(URDF): adjust joint positionGain ⚙️chore(Python): update camera offsets; adjust tag detection orientation

File: 96wellplate.urdf (robot description, URDF)
Before this commit: robot stl_object, 1 links, 0 joints
Links:
- link base_link: geometry collision mesh filename=parts-meshes/96wellplate0.stl scale=0.001 0.001 0.001; visual mesh filename=parts-meshes/96wellplate0.stl scale=0.001 0.001 0.001

File: dorna2-rebuild/urdf/dorna2-rebuild copy.urdf (robot description, URDF)
Before this commit: robot dorna2-rebuild, 7 links, 6 joints
Links:
- link wrist2: geometry collision mesh filename=package://dorna2-rebuild/meshes/wrist2.STL; visual mesh filename=package://dorna2-rebuild/meshes/wrist2.STL
